File: pcb/live-caption-badge.kicad_pcb (KiCad board)
At the start: 4 copper layers, 170 x 105.1 mm, 123 parts, among them J1 Conn_01x24, J2 Conn_01x06, J4 AudioJack4, J5 USB_C_Receptacle_USB2.0_16P, Q1 Si1308EDL, Q2 SS8050, Q3 SS8050, SW1 SW_DPDT_x2, SW2 RST, SW3 BTN, SW4 BTN, SW5 BTN, SW6 FLASH, U1 ESP32-S3-WROOM-1, U2 HE9073A33M5R, U3 HE9073A33M5R, U4 ES7210, U5 ES8311, U6 IS31AP2005

Commit message: pcb: rev 2 ready?
Parts:
- removed the REF** at (35.0, 110.0)
- added C48: 22pF, Capacitor_SMD:C_0603_1608Metric, F.Cu at (187.0, 68.0)
- moved J2 47.9 mm to (80.0, 75.0)
Routing:
- net /UART_TX: track 15.0 -> 65.5 mm, vias 0 -> 1
- net /UART_RX: track 18.1 -> 64.2 mm, vias 0 -> 1
- net /UART_DTR: track 13.5 -> 57.9 mm, vias 1 -> 3
- net /UART_RTS: track 22.6 -> 55.6 mm
- net /ESP_~{EN}: track 87.4 -> 81.9 mm
- net /Audio/MIC_IN: track 40.7 -> 37.7 mm
- net GNDA: track 19.3 -> 16.8 mm, vias 6 -> 5
- net /Audio/AUDIO_OUT: track 53.2 -> 51.0 mm
- net VBUS: track 58.5 -> 57.8 mm
Other:
- board text added: "LIVE CAPTION BADGE"
- board text added: "REV 2 EECS 473 FA 2024"
- board text added: "pain"
- board text removed: "LIVE CAPTION BADGE REV 2 EECS 473 FA 2024"
